File: Kretsskjema/IELET2111.kicad_sch (KiCad schematic)
At the start: 32 parts, among them J1 Screw_Terminal_01x04, J2 Screw_Terminal_01x05, Q1 BP103BF, Q2 BP103BF, SW1 SW_DIP_x04, U1 V7805-1000, U2 D168K

Commit message: Endringer på kicad filer
Connections:
- net +5V: no longer J1.4 (Pin_4)
- new net +12V: J1.4 (Pin_4)
Changed lines of the file:
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@@
-    )
-  )
-  (symbol (lib_id "power:+5V") (at 68.58 69.85 0) (unit 1)
-    (in_bom yes) (on_board yes) (dnp no) (fields_autoplaced)
-    (property "Reference" "#PWR010" (at 68.58 73.66 0)
-      (effects (font (size 1.27 1.27)) hide)
-    )
-    (property "Value" "+5V" (at 68.58 66.04 0)
-      (effects (font (size 1.27 1.27)))
-    )
-    (property "Footprint" "" (at 68.58 69.85 0)
-      (effects (font (size 1.27 1.27)) hide)
-    )
-    (property "Datasheet" "" (at 68.58 69.85 0)
-      (effects (font (size 1.27 1.27)) hide)
-    )
-    (pin "1")
-    (instances
-      (project "IELET2111"
-        (path "/90cbe6da-ff6a-49ba-8970-f65a4915c5f7"
-          (reference "#PWR010") (unit 1)
-        )
-      )
     )
   )
@@
         )
       )
+    )
+  )
+  (symbol (lib_id "power:+12V") (at 68.58 69.85 0) (unit 1)
+    (in_bom yes) (on_board yes) (dnp no) (fields_autoplaced)
+    (property "Reference" "#PWR010" (at 68.58 73.66 0)
+      (effects (font (size 1.27 1.27)) hide)
+    )
+    (property "Value" "+12V" (at 68.58 66.04 0)
+      (effects (font (size 1.27 1.27)))
+    )
+    (property "Footprint" "" (at 68.58 69.85 0)
+      (effects (font (size 1.27 1.27)) hide)
+    )
+    (property "Datasheet" "" (at 68.58 69.85 0)
+      (effects (font (size 1.27 1.27)) hide)
+    )
+    (pin "1")
+    (instances
+      (project "IELET2111"
+        (path "/90cbe6da-ff6a-49ba-8970-f65a4915c5f7"
+          (reference "#PWR010") (unit 1)
+        )
+      )
